File: pcb/power/rgbLedDriver.sch (KiCad schematic (older format))
At the start: 39 parts, among them Q1 MMBT3904, Q2 MMBT3904, Q3 MMBT3904, Q4 MMBT3904, Q5 MMBT3904, Q6 MMBT3904, Q7 DMG2305UX, Q8 DMG2305UX, Q9 DMG2305UX

Commit message: Almost done with the schematics. Some fine tuning is left.
Parts:
- renumbered C4 to C11, C5 to C12, C1 to C13, C6 to C14, C7 to C15, C2 to C16, C8 to C17, C9 to C18, C3 to C19, D1 to D5, D5 to D6, D2 to D7, D6 to D8, L2 to L3, L3 to L4, L1 to L5, Q6 to Q4, Q4 to Q5, Q5 to Q6, Q8 to Q7, Q7 to Q8, R11 to R18, R12 to R19, R1 to R20, R13 to R21, R14 to R22, R2 to R23, R15 to R24, R16 to R25, R3 to R26, R17 to R27, R18 to R28, R4 to R29
Changed lines of the file:
@@
 $Descr A4 11693 8268
 encoding utf-8
-Sheet 2 4
+Sheet 2 2
 Title "RGB LED Driver"
 Date "2016-11-27"
@@
 $EndDescr
 $Comp
-L D D1
+L D D5
 U 1 1 5837550B
 P 3400 6300
-F 0 "D1" V 3450 6150 50  0000 C CNN
+F 0 "D5" V 3450 6150 50  0000 C CNN
 F 1 "1N4148WFL-G" V 3350 5950 50  0000 C CNN
 F 2 "" H 3400 6300 50  0000 C CNN
@@
 $EndComp
 $Comp
-L R R2
+L R R23
 U 1 1 58375629
 P 2600 5600
-F 0 "R2" V 2680 5600 50  0000 C CNN
+F 0 "R23" V 2680 5600 50  0000 C CNN
 F 1 "10k" V 2600 5600 50  0000 C CNN
 F 2 "" V 2530 5600 50  0000 C CNN
@@
 $EndComp
 $Comp
-L R R1
+L R R20
 U 1 1 5837574C
 P 2000 6750
-F 0 "R1" V 2080 6750 50  0000 C CNN
+F 0 "R20" V 2080 6750 50  0000 C CNN
 F 1 "470R" V 2000 6750 50  0000 C CNN
 F 2 "" V 1930 6750 50  0000 C CNN
@@
 $EndComp
 $Comp
-L C C1
+L C C13
 U 1 1 5837578D
 P 2000 6450
-F 0 "C1" H 2025 6550 50  0000 L CNN
+F 0 "C13" H 2025 6550 50  0000 L CNN
 F 1 "150p" H 2025 6350 50  0000 L CNN
 F 2 "" H 2038 6300 50  0000 C CNN
@@
 PWM_G
 $Comp
-L INDUCTOR L1
+L INDUCTOR L5
 U 1 1 58375D14
 P 4150 6200
-F 0 "L1" V 4350 6200 50  0000 C CNN
+F 0 "L5" V 4350 6200 50  0000 C CNN
 F 1 "33u" V 4250 6200 50  0000 C CNN
 F 2 "" H 4150 6200 50  0000 C CNN
@@
 $EndComp
 $Comp
-L C C2
+L C C16
 U 1 1 58375E8F
 P 4550 6600
-F 0 "C2" H 4575 6700 50  0000 L CNN
+F 0 "C16" H 4575 6700 50  0000 L CNN
 F 1 "10u" H 4575 6500 50  0000 L CNN
 F 2 "" H 4588 6450 50  0000 C CNN
@@
 LED_G_N
 $Comp
-L R R3
+L R R26
 U 1 1 5837686D
 P 4850 6850
-F 0 "R3" V 4930 6850 50  0000 C CNN
+F 0 "R26" V 4930 6850 50  0000 C CNN
 F 1 "0.1R" V 4850 6850 50  0000 C CNN
 F 2 "" V 4780 6850 50  0000 C CNN
@@
 $EndComp
 $Comp
-L C C3
+L C C19
 U 1 1 583772C0
 P 5600 6850
-F 0 "C3" H 5625 6950 50  0000 L CNN
+F 0 "C19" H 5625 6950 50  0000 L CNN
 F 1 "22n" H 5625 6750 50  0000 L CNN
 F 2 "" H 5638 6700 50  0000 C CNN
@@
 $EndComp
 $Comp
-L R R4
+L R R29
 U 1 1 5837748D
 P 5250 6650
-F 0 "R4" V 5330 6650 50  0000 C CNN
+F 0 "R29" V 5330 6650 50  0000 C CNN
 F 1 "4.7k" V 5250 6650 50  0000 C CNN
 F 2 "" V 5180 6650 50  0000 C CNN
@@
 Connection ~ 5600 6650
 $Comp
-L R R14
+L R R22
 U 1 1 5837BEFE
 P 2600 3400
-F 0 "R14" V 2680 3400 50  0000 C CNN
+F 0 "R22" V 2680 3400 50  0000 C CNN
 F 1 "10k" V 2600 3400 50  0000 C CNN
 F 2 "" V 2530 3400 50  0000 C CNN
@@
 $EndComp
 $Comp
-L R R12
+L R R19
 U 1 1 5837BF05
 P 2000 4550
-F 0 "R12" V 2080 4550 50  0000 C CNN
+F 0 "R19" V 2080 4550 50  0000 C CNN
 F 1 "470R" V 2000 4550 50  0000 C CNN
 F 2 "" V 1930 4550 50  0000 C CNN
@@
 $EndComp
 $Comp
-L C C5
+L C C12
 U 1 1 5837BF0C
 P 2000 4250
-F 0 "C5" H 2025 4350 50  0000 L CNN
+F 0 "C12" H 2025 4350 50  0000 L CNN
 F 1 "150p" H 2025 4150 50  0000 L CNN
 F 2 "" H 2038 4100 50  0000 C CNN
@@
 PWM_B
 $Comp
-L INDUCTOR L3
+L INDUCTOR L4
 U 1 1 5837BF14
 P 4150 4000
-F 0 "L3" V 4350 4000 50  0000 C CNN
+F 0 "L4" V 4350 4000 50  0000 C CNN
 F 1 "33u" V 4250 4000 50  0000 C CNN
 F 2 "" H 4150 4000 50  0000 C CNN
@@
 $EndComp
 $Comp
-L C C7
+L C C15
 U 1 1 5837BF22
 P 4550 4400
-F 0 "C7" H 4575 4500 50  0000 L CNN
+F 0 "C15" H 4575 4500 50  0000 L CNN
 F 1 "10u" H 4575 4300 50  0000 L CNN
 F 2 "" H 4588 4250 50  0000 C CNN
@@
 LED_B_N
 $Comp
-L R R16
+L R R25
 U 1 1 5837BF2B
 P 4850 4650
-F 0 "R16" V 4930 4650 50  0000 C CNN
+F 0 "R25" V 4930 4650 50  0000 C CNN
 F 1 "0.1R" V 4850 4650 50  0000 C CNN
 F 2 "" V 4780 4650 50  0000 C CNN
@@
 $EndComp
 $Comp
-L C C9
+L C C18
 U 1 1 5837BF32
 P 5600 4650
-F 0 "C9" H 5625 4750 50  0000 L CNN
+F 0 "C18" H 5625 4750 50  0000 L CNN
 F 1 "22n" H 5625 4550 50  0000 L CNN
 F 2 "" H 5638 4500 50  0000 C CNN
@@
 $EndComp
 $Comp
-L R R18
+L R R28
 U 1 1 5837BF39
 P 5250 4450
-F 0 "R18" V 5330 4450 50  0000 C CNN
+F 0 "R28" V 5330 4450 50  0000 C CNN
 F 1 "4.7k" V 5250 4450 50  0000 C CNN
 F 2 "" V 5180 4450 50  0000 C CNN
@@
 Connection ~ 5600 4450
 $Comp
-L Q_NPN_BCE Q6
+L Q_NPN_BCE Q4
 U 1 1 5837C3ED
 P 2850 1650
-F 0 "Q6" H 3100 1750 50  0000 R CNN
+F 0 "Q4" H 3100 1750 50  0000 R CNN
 F 1 "MMBT3904" H 3400 1550 50  0000 R CNN
 F 2 "" H 3050 1750 50  0000 C CNN
@@
 $EndComp
 $Comp
-L Q_PMOS_DGS Q8
+L Q_PMOS_DGS Q7
 U 1 1 5837C3F4
 P 3400 1200
-F 0 "Q8" V 3600 1100 50  0000 R CNN
+F 0 "Q7" V 3600 1100 50  0000 R CNN
 F 1 "DMG2305UX" V 3350 1100 50  0000 R CNN
 F 2 "" H 3600 1300 50  0000 C CNN
@@
 $EndComp
 $Comp
-L R R13
+L R R21
 U 1 1 5837C403
 P 2600 1350
-F 0 "R13" V 2680 1350 50  0000 C CNN
+F 0 "R21" V 2680 1350 50  0000 C CNN
 F 1 "10k" V 2600 1350 50  0000 C CNN
 F 2 "" V 2530 1350 50  0000 C CNN
@@
 $EndComp
 $Comp
-L R R11
+L R R18
 U 1 1 5837C40A
 P 2000 2500
-F 0 "R11" V 2080 2500 50  0000 C CNN
+F 0 "R18" V 2080 2500 50  0000 C CNN
 F 1 "470R" V 2000 2500 50  0000 C CNN
 F 2 "" V 1930 2500 50  0000 C CNN
@@
 $EndComp
 $Comp
-L C C4
+L C C11
 U 1 1 5837C411
 P 2000 2200
-F 0 "C4" H 2025 2300 50  0000 L CNN
+F 0 "C11" H 2025 2300 50  0000 L CNN
 F 1 "150p" H 2025 2100 50  0000 L CNN
 F 2 "" H 2038 2050 50  0000 C CNN
@@
 PWM_R
 $Comp
-L INDUCTOR L2
+L INDUCTOR L3
 U 1 1 5837C419
 P 4150 1950
-F 0 "L2" V 4100 1950 50  0000 C CNN
+F 0 "L3" V 4100 1950 50  0000 C CNN
 F 1 "33u" V 4250 1950 50  0000 C CNN
 F 2 "" H 4150 1950 50  0000 C CNN
@@
 $EndComp
 $Comp
-L D_Schottky D5
+L D_Schottky D6
 U 1 1 5837C420
 P 3750 2350
-F 0 "D5" V 3700 2500 50  0000 C CNN
+F 0 "D6" V 3700 2500 50  0000 C CNN
 F 1 "VS-10MQ060NPbF" V 3800 2800 50  0000 C CNN
 F 2 "" H 3750 2350 50  0000 C CNN
@@
 $EndComp
 $Comp
-L C C6
+L C C14
 U 1 1 5837C427
 P 4550 2350
-F 0 "C6" H 4575 2450 50  0000 L CNN
+F 0 "C14" H 4575 2450 50  0000 L CNN
 F 1 "10u" H 4575 2250 50  0000 L CNN
 F 2 "" H 4588 2200 50  0000 C CNN
@@
 LED_R_N
 $Comp
-L R R15
+L R R24
 U 1 1 5837C430
 P 4850 2600
-F 0 "R15" V 4930 2600 50  0000 C CNN
+F 0 "R24" V 4930 2600 50  0000 C CNN
 F 1 "0.1R" V 4850 2600 50  0000 C CNN
 F 2 "" V 4780 2600 50  0000 C CNN
@@
 $EndComp
 $Comp
-L C C8
+L C C17
 U 1 1 5837C437
 P 5600 2600
-F 0 "C8" H 5625 2700 50  0000 L CNN
+F 0 "C17" H 5625 2700 50  0000 L CNN
 F 1 "22n" H 5625 2500 50  0000 L CNN
 F 2 "" H 5638 2450 50  0000 C CNN
@@
 $EndComp
 $Comp
-L R R17
+L R R27
 U 1 1 5837C43E
 P 5250 2400
-F 0 "R17" V 5330 2400 50  0000 C CNN
+F 0 "R27" V 5330 2400 50  0000 C CNN
 F 1 "4.7k" V 5250 2400 50  0000 C CNN
 F 2 "" V 5180 2400 50  0000 C CNN
@@
 $EndComp
 $Comp
-L Q_PMOS_DGS Q7
+L Q_PMOS_DGS Q8
 U 1 1 583C6F4A
 P 3400 3250
-F 0 "Q7" V 3600 3150 50  0000 R CNN
+F 0 "Q8" V 3600 3150 50  0000 R CNN
 F 1 "DMG2305UX" V 3350 3150 50  0000 R CNN
 F 2 "" H 3600 3350 50  0000 C CNN
@@
 $EndComp
 $Comp
-L Q_NPN_BCE Q4
+L Q_NPN_BCE Q5
 U 1 1 583C7003
 P 2850 3700
-F 0 "Q4" H 3100 3800 50  0000 R CNN
+F 0 "Q5" H 3100 3800 50  0000 R CNN
 F 1 "MMBT3904" H 3400 3600 50  0000 R CNN
 F 2 "" H 3050 3800 50  0000 C CNN
@@
 $EndComp
 $Comp
-L Q_NPN_BCE Q5
+L Q_NPN_BCE Q6
 U 1 1 583C75B3
 P 2850 5900
-F 0 "Q5" H 3100 6000 50  0000 R CNN
+F 0 "Q6" H 3100 6000 50  0000 R CNN
 F 1 "MMBT3904" H 3400 5800 50  0000 R CNN
 F 2 "" H 3050 6000 50  0000 C CNN
@@
 $EndComp
 $Comp
-L D_Schottky D2
+L D_Schottky D7
 U 1 1 583CD480
 P 3750 4400
-F 0 "D2" V 3700 4550 50  0000 C CNN
+F 0 "D7" V 3700 4550 50  0000 C CNN
 F 1 "VS-10MQ060NPbF" V 3800 4850 50  0000 C CNN
 F 2 "" H 3750 4400 50  0000 C CNN
@@
 $EndComp
 $Comp
-L D_Schottky D6
+L D_Schottky D8
 U 1 1 583CD596
 P 3750 6600
-F 0 "D6" V 3700 6750 50  0000 C CNN
+F 0 "D8" V 3700 6750 50  0000 C CNN
 F 1 "VS-10MQ060NPbF" V 3800 7050 50  0000 C CNN
 F 2 "" H 3750 6600 50  0000 C CNN

Commit message: Finished schematics.
Parts:
- renumbered C11 to C12, C12 to C13, C13 to C14, C14 to C15, C15 to C16, C16 to C17, C17 to C18, C18 to C19, C19 to C20, D7 to D10, D8 to D11, D3 to D6, D4 to D7, D5 to D8, D6 to D9, R18 to R21, R19 to R22, R20 to R23, R21 to R24, R22 to R25, R23 to R26, R24 to R27, R25 to R28, R26 to R29, R27 to R30, R28 to R31, R29 to R32
Connections:
- no-connect marks 1 -> 0
Changed lines of the file:
@@
 encoding utf-8
 Sheet 2 2
-Title "RGB LED Driver"
-Date "2016-11-27"
+Title "RGB LED Driver "
+Date "2016-12-01"
 Rev "1.0"
-Comp ""
-Comment1 ""
+Comp "Uppsala University"
+Comment1 "Project: Swakeup"
 Comment2 ""
 Comment3 ""
@@
 $EndDescr
 $Comp
-L D D5
+L D D8
 U 1 1 5837550B
 P 3400 6300
-F 0 "D5" V 3450 6150 50  0000 C CNN
+F 0 "D8" V 3450 6150 50  0000 C CNN
 F 1 "1N4148WFL-G" V 3350 5950 50  0000 C CNN
 F 2 "" H 3400 6300 50  0000 C CNN
@@
 $EndComp
 $Comp
-L R R23
+L R R26
 U 1 1 58375629
 P 2600 5600
-F 0 "R23" V 2680 5600 50  0000 C CNN
+F 0 "R26" V 2680 5600 50  0000 C CNN
 F 1 "10k" V 2600 5600 50  0000 C CNN
 F 2 "" V 2530 5600 50  0000 C CNN
@@
 $EndComp
 $Comp
-L R R20
+L R R23
 U 1 1 5837574C
 P 2000 6750
-F 0 "R20" V 2080 6750 50  0000 C CNN
+F 0 "R23" V 2080 6750 50  0000 C CNN
 F 1 "470R" V 2000 6750 50  0000 C CNN
 F 2 "" V 1930 6750 50  0000 C CNN
@@
 $EndComp
 $Comp
-L C C13
+L C C14
 U 1 1 5837578D
 P 2000 6450
-F 0 "C13" H 2025 6550 50  0000 L CNN
+F 0 "C14" H 2025 6550 50  0000 L CNN
 F 1 "150p" H 2025 6350 50  0000 L CNN
 F 2 "" H 2038 6300 50  0000 C CNN
@@
 $EndComp
 $Comp
-L C C16
+L C C17
 U 1 1 58375E8F
 P 4550 6600
-F 0 "C16" H 4575 6700 50  0000 L CNN
+F 0 "C17" H 4575 6700 50  0000 L CNN
 F 1 "10u" H 4575 6500 50  0000 L CNN
 F 2 "" H 4588 6450 50  0000 C CNN
@@
 LED_G_N
 $Comp
-L R R26
+L R R29
 U 1 1 5837686D
 P 4850 6850
-F 0 "R26" V 4930 6850 50  0000 C CNN
+F 0 "R29" V 4930 6850 50  0000 C CNN
 F 1 "0.1R" V 4850 6850 50  0000 C CNN
 F 2 "" V 4780 6850 50  0000 C CNN
@@
 $EndComp
 $Comp
-L C C19
+L C C20
 U 1 1 583772C0
 P 5600 6850
-F 0 "C19" H 5625 6950 50  0000 L CNN
+F 0 "C20" H 5625 6950 50  0000 L CNN
 F 1 "22n" H 5625 6750 50  0000 L CNN
 F 2 "" H 5638 6700 50  0000 C CNN
@@
 $EndComp
 $Comp
-L R R29
+L R R32
 U 1 1 5837748D
 P 5250 6650
-F 0 "R29" V 5330 6650 50  0000 C CNN
+F 0 "R32" V 5330 6650 50  0000 C CNN
 F 1 "4.7k" V 5250 6650 50  0000 C CNN
 F 2 "" V 5180 6650 50  0000 C CNN
@@
 Connection ~ 5600 6650
 $Comp
-L R R22
+L R R25
 U 1 1 5837BEFE
 P 2600 3400
-F 0 "R22" V 2680 3400 50  0000 C CNN
+F 0 "R25" V 2680 3400 50  0000 C CNN
 F 1 "10k" V 2600 3400 50  0000 C CNN
 F 2 "" V 2530 3400 50  0000 C CNN
@@
 $EndComp
 $Comp
-L R R19
+L R R22
 U 1 1 5837BF05
 P 2000 4550
-F 0 "R19" V 2080 4550 50  0000 C CNN
+F 0 "R22" V 2080 4550 50  0000 C CNN
 F 1 "470R" V 2000 4550 50  0000 C CNN
 F 2 "" V 1930 4550 50  0000 C CNN
@@
 $EndComp
 $Comp
-L C C12
+L C C13
 U 1 1 5837BF0C
 P 2000 4250
-F 0 "C12" H 2025 4350 50  0000 L CNN
+F 0 "C13" H 2025 4350 50  0000 L CNN
 F 1 "150p" H 2025 4150 50  0000 L CNN
 F 2 "" H 2038 4100 50  0000 C CNN
@@
 $EndComp
 $Comp
-L C C15
+L C C16
 U 1 1 5837BF22
 P 4550 4400
-F 0 "C15" H 4575 4500 50  0000 L CNN
+F 0 "C16" H 4575 4500 50  0000 L CNN
 F 1 "10u" H 4575 4300 50  0000 L CNN
 F 2 "" H 4588 4250 50  0000 C CNN
@@
 LED_B_N
 $Comp
-L R R25
+L R R28
 U 1 1 5837BF2B
 P 4850 4650
-F 0 "R25" V 4930 4650 50  0000 C CNN
+F 0 "R28" V 4930 4650 50  0000 C CNN
 F 1 "0.1R" V 4850 4650 50  0000 C CNN
 F 2 "" V 4780 4650 50  0000 C CNN
@@
 $EndComp
 $Comp
-L C C18
+L C C19
 U 1 1 5837BF32
 P 5600 4650
-F 0 "C18" H 5625 4750 50  0000 L CNN
+F 0 "C19" H 5625 4750 50  0000 L CNN
 F 1 "22n" H 5625 4550 50  0000 L CNN
 F 2 "" H 5638 4500 50  0000 C CNN
@@
 $EndComp
 $Comp
-L R R28
+L R R31
 U 1 1 5837BF39
 P 5250 4450
-F 0 "R28" V 5330 4450 50  0000 C CNN
+F 0 "R31" V 5330 4450 50  0000 C CNN
 F 1 "4.7k" V 5250 4450 50  0000 C CNN
 F 2 "" V 5180 4450 50  0000 C CNN
@@
 $EndComp
 $Comp
-L R R21
+L R R24
 U 1 1 5837C403
 P 2600 1350
-F 0 "R21" V 2680 1350 50  0000 C CNN
+F 0 "R24" V 2680 1350 50  0000 C CNN
 F 1 "10k" V 2600 1350 50  0000 C CNN
 F 2 "" V 2530 1350 50  0000 C CNN
@@
 $EndComp
 $Comp
-L R R18
+L R R21
 U 1 1 5837C40A
 P 2000 2500
-F 0 "R18" V 2080 2500 50  0000 C CNN
+F 0 "R21" V 2080 2500 50  0000 C CNN
 F 1 "470R" V 2000 2500 50  0000 C CNN
 F 2 "" V 1930 2500 50  0000 C CNN
@@
 $EndComp
 $Comp
-L C C11
+L C C12
 U 1 1 5837C411
 P 2000 2200
-F 0 "C11" H 2025 2300 50  0000 L CNN
+F 0 "C12" H 2025 2300 50  0000 L CNN
 F 1 "150p" H 2025 2100 50  0000 L CNN
 F 2 "" H 2038 2050 50  0000 C CNN
@@
 $EndComp
 $Comp
-L D_Schottky D6
+L D_Schottky D9
 U 1 1 5837C420
 P 3750 2350
-F 0 "D6" V 3700 2500 50  0000 C CNN
+F 0 "D9" V 3700 2500 50  0000 C CNN
 F 1 "VS-10MQ060NPbF" V 3800 2800 50  0000 C CNN
 F 2 "" H 3750 2350 50  0000 C CNN
@@
 $EndComp
 $Comp
-L C C14
+L C C15
 U 1 1 5837C427
 P 4550 2350
-F 0 "C14" H 4575 2450 50  0000 L CNN
+F 0 "C15" H 4575 2450 50  0000 L CNN
 F 1 "10u" H 4575 2250 50  0000 L CNN
 F 2 "" H 4588 2200 50  0000 C CNN
@@
 LED_R_N
 $Comp
-L R R24
+L R R27
 U 1 1 5837C430
 P 4850 2600
-F 0 "R24" V 4930 2600 50  0000 C CNN
+F 0 "R27" V 4930 2600 50  0000 C CNN
 F 1 "0.1R" V 4850 2600 50  0000 C CNN
 F 2 "" V 4780 2600 50  0000 C CNN
@@
 $EndComp
 $Comp
-L C C17
+L C C18
 U 1 1 5837C437
 P 5600 2600
-F 0 "C17" H 5625 2700 50  0000 L CNN
+F 0 "C18" H 5625 2700 50  0000 L CNN
 F 1 "22n" H 5625 2500 50  0000 L CNN
 F 2 "" H 5638 2450 50  0000 C CNN
@@
 $EndComp
 $Comp
-L R R27
+L R R30
 U 1 1 5837C43E
 P 5250 2400
-F 0 "R27" V 5330 2400 50  0000 C CNN
+F 0 "R30" V 5330 2400 50  0000 C CNN
 F 1 "4.7k" V 5250 2400 50  0000 C CNN
 F 2 "" V 5180 2400 50  0000 C CNN
@@
 Connection ~ 5600 2400
 Connection ~ 1050 1100
-NoConn ~ 7900 3350
 Text HLabel 950  1100 0    60   Input ~ 0
 V20
@@
 fcutt,off=1.539 kHz
 $Comp
-L D D4
+L D D7
 U 1 1 583CC236
 P 3400 4100
-F 0 "D4" V 3450 3950 50  0000 C CNN
+F 0 "D7" V 3450 3950 50  0000 C CNN
 F 1 "1N4148WFL-G" V 3350 3750 50  0000 C CNN
 F 2 "" H 3400 4100 50  0000 C CNN
@@
 $EndComp
 $Comp
-L D D3
+L D D6
 U 1 1 583CC52C
 P 3400 2050
-F 0 "D3" V 3450 1900 50  0000 C CNN
+F 0 "D6" V 3450 1900 50  0000 C CNN
 F 1 "1N4148WFL-G" V 3350 1700 50  0000 C CNN
 F 2 "" H 3400 2050 50  0000 C CNN
@@
 $EndComp
 $Comp
-L D_Schottky D7
+L D_Schottky D10
 U 1 1 583CD480
 P 3750 4400
-F 0 "D7" V 3700 4550 50  0000 C CNN
+F 0 "D10" V 3700 4550 50  0000 C CNN
 F 1 "VS-10MQ060NPbF" V 3800 4850 50  0000 C CNN
 F 2 "" H 3750 4400 50  0000 C CNN
@@
 $EndComp
 $Comp
-L D_Schottky D8
+L D_Schottky D11
 U 1 1 583CD596
 P 3750 6600
-F 0 "D8" V 3700 6750 50  0000 C CNN
+F 0 "D11" V 3700 6750 50  0000 C CNN
 F 1 "VS-10MQ060NPbF" V 3800 7050 50  0000 C CNN
 F 2 "" H 3750 6600 50  0000 C CNN
