File: pcb/power/rgbLedDriver.sch (KiCad schematic (older format))
At the start: 39 parts, among them Q1 MMBT3904, Q2 MMBT3904, Q3 MMBT3904, Q4 MMBT3904, Q5 MMBT3904, Q6 MMBT3904, Q7 DMG2305UX, Q8 DMG2305UX, Q9 DMG2305UX

Commit message: Fixed the board. This is rev 2.
Parts:
- removed Q1, Q2, Q3, Q4, Q5, Q6: MMBT3904, TO_SOT_Packages_SMD:SOT-23_Handsoldering, symbol Q_NPN_BCE
- removed Q7, Q8, Q9: DMG2305UX, TO_SOT_Packages_SMD:SOT-23_Handsoldering, symbol Q_PMOS_DGS
- added Q1, Q2, Q3, Q4, Q5, Q6: MMBT3904, TO_SOT_Packages_SMD:SOT-23, symbol MMBT3904
- added Q7, Q8, Q9: DMG2305UX, TO_SOT_Packages_SMD:SOT-23, symbol DMG2305UX
Connections:
- net GND: now also Q1.2 (E), Q2.2 (E), Q3.2 (E)
- net V20: now also Q4.3 (C), Q5.3 (C), Q6.3 (C), Q7.2 (S), Q8.2 (S), Q9.2 (S)
- net at D6.1 (K), R24.1: now also Q1.3 (C), Q4.1 (B)
- net at D6.2 (A): now also Q4.2 (E), Q7.1 (G)
- net at D9.1 (K), L3.1: now also Q7.3 (D)
- net at C12.1, R21.1: now also Q1.1 (B)
- net at C13.1, R22.1: now also Q2.1 (B)
- net at C14.1, R23.1: now also Q3.1 (B)
- net at D8.1 (K), R26.1: now also Q3.3 (C), Q6.1 (B)
- net at D7.1 (K), R25.1: now also Q2.3 (C), Q5.1 (B)
- net at D7.2 (A): now also Q5.2 (E), Q8.1 (G)
- net at D10.1 (K), L4.1: now also Q8.3 (D)
- net at D8.2 (A): now also Q6.2 (E), Q9.1 (G)
- net at D11.1 (K), L5.1: now also Q9.3 (D)
Changed lines of the file:
@@
 OPAMP_B_P
-$Comp
-L Q_PMOS_DGS Q7
-U 1 1 5837C3F4
-P 3400 1200
-F 0 "Q7" V 3600 1100 50  0000 R CNN
-F 1 "DMG2305UX" V 3350 1100 50  0000 R CNN
-F 2 "TO_SOT_Packages_SMD:SOT-23_Handsoldering" H 3600 1300 50  0001 C CNN
-F 3 "http://www.diodes.com/_files/datasheets/DMG2305UX.pdf" H 3400 1200 50  0001 C CNN
-F 4 "DMG2305UX-13DICT-ND" H 3400 1200 60  0001 C CNN "Digikey"
-	1    3400 1200
-	0    -1   -1   0
-$EndComp
 $Comp
 L R R24
@@
 F 1 "VS-10MQ060NPbF" V 3800 2800 50  0000 C CNN
 F 2 "Diodes_SMD:SMA_Handsoldering" H 3750 2350 50  0001 C CNN
-F 3 "http://www.vishay.com/docs/88869/packaging.pdf" H 3750 2350 50  0001 C CNN
+F 3 "http://www.vishay.com/docs/94118/vs-10mq060npbf.pdf" H 3750 2350 50  0001 C CNN
 F 4 "10MQ060NPBFCT-ND" V 3800 2950 60  0001 C CNN "Digikey"
 	1    3750 2350
@@
 $EndComp
 $Comp
-L Q_PMOS_DGS Q8
-U 1 1 5841A28D
-P 3400 3250
-F 0 "Q8" V 3600 3150 50  0000 R CNN
-F 1 "DMG2305UX" V 3350 3150 50  0000 R CNN
-F 2 "TO_SOT_Packages_SMD:SOT-23_Handsoldering" H 3600 3350 50  0001 C CNN
-F 3 "http://www.diodes.com/_files/datasheets/DMG2305UX.pdf" H 3400 3250 50  0001 C CNN
-F 4 "DMG2305UX-13DICT-ND" H 3400 3250 60  0001 C CNN "Digikey"
-	1    3400 3250
-	0    -1   -1   0
-$EndComp
-$Comp
-L Q_PMOS_DGS Q9
-U 1 1 5841A571
-P 3400 5450
-F 0 "Q9" V 3600 5350 50  0000 R CNN
-F 1 "DMG2305UX" V 3350 5350 50  0000 R CNN
-F 2 "TO_SOT_Packages_SMD:SOT-23_Handsoldering" H 3600 5550 50  0001 C CNN
-F 3 "http://www.diodes.com/_files/datasheets/DMG2305UX.pdf" H 3400 5450 50  0001 C CNN
-F 4 "DMG2305UX-13DICT-ND" H 3400 5450 60  0001 C CNN "Digikey"
-	1    3400 5450
-	0    -1   -1   0
-$EndComp
-$Comp
-L Q_NPN_BCE Q4
-U 1 1 5837C3ED
-P 2850 1650
-F 0 "Q4" H 3100 1750 50  0000 R CNN
-F 1 "MMBT3904" H 3400 1550 50  0000 R CNN
-F 2 "TO_SOT_Packages_SMD:SOT-23_Handsoldering" H 3050 1750 50  0001 C CNN
-F 3 "http://www.mccsemi.com/up_pdf/MMBT3904(SOT-23).pdf" H 2850 1650 50  0001 C CNN
-F 4 "MMBT3904TPMSCT-ND" H 3550 1600 60  0001 C CNN "Digikey"
-	1    2850 1650
-	1    0    0    -1
-$EndComp
-$Comp
-L Q_NPN_BCE Q5
-U 1 1 5841AE74
-P 2850 3700
-F 0 "Q5" H 3100 3800 50  0000 R CNN
-F 1 "MMBT3904" H 3400 3600 50  0000 R CNN
-F 2 "TO_SOT_Packages_SMD:SOT-23_Handsoldering" H 3050 3800 50  0001 C CNN
-F 3 "http://www.mccsemi.com/up_pdf/MMBT3904(SOT-23).pdf" H 2850 3700 50  0001 C CNN
-F 4 "MMBT3904TPMSCT-ND" H 3550 3650 60  0001 C CNN "Digikey"
-	1    2850 3700
-	1    0    0    -1
-$EndComp
-$Comp
-L Q_NPN_BCE Q6
-U 1 1 5841B110
-P 2850 5900
-F 0 "Q6" H 3100 6000 50  0000 R CNN
-F 1 "MMBT3904" H 3400 5800 50  0000 R CNN
-F 2 "TO_SOT_Packages_SMD:SOT-23_Handsoldering" H 3050 6000 50  0001 C CNN
-F 3 "http://www.mccsemi.com/up_pdf/MMBT3904(SOT-23).pdf" H 2850 5900 50  0001 C CNN
-F 4 "MMBT3904TPMSCT-ND" H 3550 5850 60  0001 C CNN "Digikey"
-	1    2850 5900
-	1    0    0    -1
-$EndComp
-$Comp
-L Q_NPN_BCE Q1
-U 1 1 5841C01A
-P 2500 2500
-F 0 "Q1" H 2750 2600 50  0000 R CNN
-F 1 "MMBT3904" H 3050 2400 50  0000 R CNN
-F 2 "TO_SOT_Packages_SMD:SOT-23_Handsoldering" H 2700 2600 50  0001 C CNN
-F 3 "http://www.mccsemi.com/up_pdf/MMBT3904(SOT-23).pdf" H 2500 2500 50  0001 C CNN
-F 4 "MMBT3904TPMSCT-ND" H 3200 2450 60  0001 C CNN "Digikey"
-	1    2500 2500
-	1    0    0    -1
-$EndComp
-$Comp
-L Q_NPN_BCE Q2
-U 1 1 5841C212
-P 2500 4550
-F 0 "Q2" H 2750 4650 50  0000 R CNN
-F 1 "MMBT3904" H 3050 4450 50  0000 R CNN
-F 2 "TO_SOT_Packages_SMD:SOT-23_Handsoldering" H 2700 4650 50  0001 C CNN
-F 3 "http://www.mccsemi.com/up_pdf/MMBT3904(SOT-23).pdf" H 2500 4550 50  0001 C CNN
-F 4 "MMBT3904TPMSCT-ND" H 3200 4500 60  0001 C CNN "Digikey"
-	1    2500 4550
-	1    0    0    -1
-$EndComp
-$Comp
-L Q_NPN_BCE Q3
-U 1 1 5841C4C0
-P 2500 6750
-F 0 "Q3" H 2750 6850 50  0000 R CNN
-F 1 "MMBT3904" H 3050 6650 50  0000 R CNN
-F 2 "TO_SOT_Packages_SMD:SOT-23_Handsoldering" H 2700 6850 50  0001 C CNN
-F 3 "http://www.mccsemi.com/up_pdf/MMBT3904(SOT-23).pdf" H 2500 6750 50  0001 C CNN
-F 4 "MMBT3904TPMSCT-ND" H 3200 6700 60  0001 C CNN "Digikey"
-	1    2500 6750
-	1    0    0    -1
-$EndComp
-$Comp
 L D D7
 U 1 1 5841D6DF
@@
 	3600 3150 3750 3150
 Wire Wire Line
-	950  1100 3200 1100
-Wire Wire Line
-	2600 1200 2600 1100
+	2600 1100 2600 1200
 Connection ~ 2600 1100
 Wire Wire Line
@@
 	2600 1650 2650 1650
 Wire Wire Line
-	2950 1450 2950 1100
+	2950 1100 2950 1450
 Connection ~ 2950 1100
 Wire Wire Line
 	2950 1850 3400 1850
-Wire Wire Line
-	3400 1400 3400 1900
 Connection ~ 3400 1850
 Wire Wire Line
@@
 	3750 1100 3750 2200
 Connection ~ 3750 1950
-Wire Wire Line
-	3600 1100 3750 1100
 Connection ~ 1050 1100
 Connection ~ 1050 3150
@@
 	5800 5500 4950 5500
 Connection ~ 4950 5700
+Wire Wire Line
+	3600 1100 3750 1100
+Wire Wire Line
+	950  1100 3200 1100
+Wire Wire Line
+	3400 1400 3400 1900
+$Comp
+L MMBT3904 Q4
+U 1 1 58A342A6
+P 2850 1650
+F 0 "Q4" H 3150 1700 50  0000 R CNN
+F 1 "MMBT3904" H 3450 1600 50  0000 R CNN
+F 2 "TO_SOT_Packages_SMD:SOT-23" H 3050 1750 50  0001 C CNN
+F 3 "http://www.mccsemi.com/up_pdf/MMBT3904(SOT-23).pdf" H 2850 1650 50  0001 C CNN
+F 4 "MMBT3904TPMSCT-ND" H 2850 1650 60  0001 C CNN "Digikey"
+	1    2850 1650
+	1    0    0    -1
+$EndComp
+$Comp
+L MMBT3904 Q1
+U 1 1 58A34880
+P 2500 2500
+F 0 "Q1" H 2800 2550 50  0000 R CNN
+F 1 "MMBT3904" H 3100 2450 50  0000 R CNN
+F 2 "TO_SOT_Packages_SMD:SOT-23" H 2700 2600 50  0001 C CNN
+F 3 "http://www.mccsemi.com/up_pdf/MMBT3904(SOT-23).pdf" H 2500 2500 50  0001 C CNN
+F 4 "MMBT3904TPMSCT-ND" H 2500 2500 60  0001 C CNN "Digikey"
+	1    2500 2500
+	1    0    0    -1
+$EndComp
+$Comp
+L MMBT3904 Q5
+U 1 1 58A34B4B
+P 2850 3700
+F 0 "Q5" H 3150 3750 50  0000 R CNN
+F 1 "MMBT3904" H 3450 3650 50  0000 R CNN
+F 2 "TO_SOT_Packages_SMD:SOT-23" H 3050 3800 50  0001 C CNN
+F 3 "http://www.mccsemi.com/up_pdf/MMBT3904(SOT-23).pdf" H 2850 3700 50  0001 C CNN
+F 4 "MMBT3904TPMSCT-ND" H 2850 3700 60  0001 C CNN "Digikey"
+	1    2850 3700
+	1    0    0    -1
+$EndComp
+$Comp
+L MMBT3904 Q2
+U 1 1 58A34E03
+P 2500 4550
+F 0 "Q2" H 2800 4600 50  0000 R CNN
+F 1 "MMBT3904" H 3100 4500 50  0000 R CNN
+F 2 "TO_SOT_Packages_SMD:SOT-23" H 2700 4650 50  0001 C CNN
+F 3 "http://www.mccsemi.com/up_pdf/MMBT3904(SOT-23).pdf" H 2500 4550 50  0001 C CNN
+F 4 "MMBT3904TPMSCT-ND" H 2500 4550 60  0001 C CNN "Digikey"
+	1    2500 4550
+	1    0    0    -1
+$EndComp
+$Comp
+L MMBT3904 Q6
+U 1 1 58A34FB5
+P 2850 5900
+F 0 "Q6" H 3150 5950 50  0000 R CNN
+F 1 "MMBT3904" H 3450 5850 50  0000 R CNN
+F 2 "TO_SOT_Packages_SMD:SOT-23" H 3050 6000 50  0001 C CNN
+F 3 "http://www.mccsemi.com/up_pdf/MMBT3904(SOT-23).pdf" H 2850 5900 50  0001 C CNN
+F 4 "MMBT3904TPMSCT-ND" H 2850 5900 60  0001 C CNN "Digikey"
+	1    2850 5900
+	1    0    0    -1
+$EndComp
+$Comp
+L MMBT3904 Q3
+U 1 1 58A35080
+P 2500 6750
+F 0 "Q3" H 2800 6800 50  0000 R CNN
+F 1 "MMBT3904" H 3100 6700 50  0000 R CNN
+F 2 "TO_SOT_Packages_SMD:SOT-23" H 2700 6850 50  0001 C CNN
+F 3 "http://www.mccsemi.com/up_pdf/MMBT3904(SOT-23).pdf" H 2500 6750 50  0001 C CNN
+F 4 "MMBT3904TPMSCT-ND" H 2500 6750 60  0001 C CNN "Digikey"
+	1    2500 6750
+	1    0    0    -1
+$EndComp
+$Comp
+L DMG2305UX Q8
+U 1 1 58A4969E
+P 3400 3250
+F 0 "Q8" V 3575 3450 50  0000 R CNN
+F 1 "DMG2305UX" V 3375 3825 50  0000 R CNN
+F 2 "TO_SOT_Packages_SMD:SOT-23" H 3600 3350 50  0001 C CNN
+F 3 "http://www.diodes.com/_files/datasheets/DMG2305UX.pdf" H 3400 3250 50  0001 C CNN
+F 4 "-" H 3400 3250 60  0001 C CNN "Digikey"
+	1    3400 3250
+	0    1    -1   0
+$EndComp
+$Comp
+L DMG2305UX Q7
+U 1 1 58A4A801
+P 3400 1200
+F 0 "Q7" V 3575 1400 50  0000 R CNN
+F 1 "DMG2305UX" V 3375 1775 50  0000 R CNN
+F 2 "TO_SOT_Packages_SMD:SOT-23" H 3600 1300 50  0001 C CNN
+F 3 "http://www.diodes.com/_files/datasheets/DMG2305UX.pdf" H 3400 1200 50  0001 C CNN
+F 4 "-" H 3400 1200 60  0001 C CNN "Digikey"
+	1    3400 1200
+	0    1    -1   0
+$EndComp
+$Comp
+L DMG2305UX Q9
+U 1 1 58A4AA57
+P 3400 5450
+F 0 "Q9" V 3575 5650 50  0000 R CNN
+F 1 "DMG2305UX" V 3375 6025 50  0000 R CNN
+F 2 "TO_SOT_Packages_SMD:SOT-23" H 3600 5550 50  0001 C CNN
+F 3 "http://www.diodes.com/_files/datasheets/DMG2305UX.pdf" H 3400 5450 50  0001 C CNN
+F 4 "-" H 3400 5450 60  0001 C CNN "Digikey"
+	1    3400 5450
+	0    1    -1   0
+$EndComp
 $EndSCHEMATC
