File: pcb/power/power.kicad_pcb (KiCad board)
At the start: 2 copper layers, 50 x 40 mm, 109 parts, among them CON1 BARREL_JACK, P1 CONN_01X04, P2 CONN_01X04, P3 CONN_01X04, P4 USB_A, P5 CONN_01X03, P6 CONN_01X03, Q1 MMBT3904, Q2 MMBT3904, Q3 MMBT3904, Q4 MMBT3904, Q5 MMBT3904, Q6 MMBT3904, Q7 DMG2305UX, Q8 DMG2305UX, Q9 DMG2305UX, U1 LM2840, U2 TS30012, U3 TPS2514ADBV, U4 LM324QT

Commit message: Finished layout.
Parts:
- removed the REF** at (152.5, 104.3)
- added G***: LOGO, Additional:UU, B.Cu at (151.1, 111.3)
- added REF**: Via_GND_04, Additional:Via_GND_06, F.Cu at (152.0, 102.9)
- added REF**: Via_GND_04, Additional:Via_GND_04, F.Cu at (163.6, 103.8)
- added REF**: Via_GND_04, Additional:Via_GND_04, F.Cu at (164.0, 105.5)
- added REF**: Via_GND_04, Additional:Via_GND_04, F.Cu at (161.7, 108.5)
- added REF**: Via_GND_04, Additional:Via_GND_04, F.Cu at (159.0, 106.9)
- added REF**: Via_GND_04, Additional:Via_GND_04, F.Cu at (158.0, 105.1)
- added REF**: Via_GND_04, Additional:Via_GND_04, F.Cu at (178.6, 117.1)
- added REF**: Via_GND_04, Additional:Via_GND_04, F.Cu at (178.6, 118.4)
- added REF**: Via_GND_04, Additional:Via_GND_04, F.Cu at (178.6, 119.8)
- added REF**: Via_GND_04, Additional:Via_GND_04, F.Cu at (154.3, 116.7)
- added REF**: Via_GND_04, Additional:Via_GND_04, F.Cu at (157.2, 116.6)
- added REF**: Via_GND_04, Additional:Via_GND_06, F.Cu at (152.9, 102.9)
- added REF**: Via_GND_04, Additional:Via_GND_04, F.Cu at (156.8, 114.9)
- added REF**: Via_GND_04, Additional:Via_GND_04, F.Cu at (156.8, 113.2)
- added REF**: Via_GND_04, Additional:Via_GND_04, F.Cu at (158.1, 112.1)
- added REF**: Via_GND_04, Additional:Via_GND_04, F.Cu at (154.7, 111.4)
- added REF**: Via_GND_04, Additional:Via_GND_04, F.Cu at (152.9, 109.6)
- added REF**: Via_GND_04, Additional:Via_GND_04, F.Cu at (155.7, 109.6)
- added REF**: Via_GND_04, Additional:Via_GND_04, F.Cu at (158.0, 110.6)
- added REF**: Via_GND_04, Additional:Via_GND_04, F.Cu at (158.0, 109.5)
- added REF**: Via_GND_04, Additional:Via_GND_04, F.Cu at (160.4, 95.8)
- added REF**: Via_GND_04, Additional:Via_GND_04, F.Cu at (160.4, 95.2)
- added REF**: Via_GND_04, Additional:Via_GND_06, F.Cu at (152.9, 102.0)
- added REF**: Via_GND_04, Additional:Via_GND_04, F.Cu at (144.4, 102.2)
- added REF**: Via_GND_04, Additional:Via_GND_04, F.Cu at (144.4, 103.5)
- added REF**: Via_GND_04, Additional:Via_GND_04, F.Cu at (144.4, 104.8)
- added REF**: Via_GND_04, Additional:Via_GND_04, F.Cu at (135.0, 107.3)
- added REF**: Via_GND_04, Additional:Via_GND_04, F.Cu at (135.0, 106.0)
- added REF**: Via_GND_04, Additional:Via_GND_04, F.Cu at (133.9, 106.0)
- added REF**: Via_GND_04, Additional:Via_GND_04, F.Cu at (133.9, 107.3)
- added REF**: Via_GND_04, Additional:Via_GND_04, F.Cu at (135.0, 92.5)
- added REF**: Via_GND_04, Additional:Via_GND_04, F.Cu at (135.0, 93.9)
- added REF**: Via_GND_04, Additional:Via_GND_04, F.Cu at (178.1, 101.5)
- added REF**: Via_GND_04, Additional:Via_GND_06, F.Cu at (152.0, 102.0)
- added REF**: Via_GND_04, Additional:Via_GND_04, F.Cu at (178.4, 101.9)
- added REF**: Via_GND_04, Additional:Via_GND_04, F.Cu at (178.4, 103.3)
- added REF**: Via_GND_1, Additional:Via_GND_1, F.Cu at (134.6, 98.0)
- added REF**: Via_GND_1, Additional:Via_GND_1, F.Cu at (134.6, 99.3)
- added REF**: Via_GND_1, Additional:Via_GND_1, F.Cu at (134.6, 100.6)
- added REF**: Via_GND_04, Additional:Via_GND_04, F.Cu at (155.3, 100.3)
- added REF**: Via_GND_1, Additional:Via_GND_1, F.Cu at (166.9, 90.9)
- added REF**: Via_GND_1, Additional:Via_GND_1, F.Cu at (165.6, 89.3)
- added REF**: Via_GND_1, Additional:Via_GND_1, F.Cu at (162.1, 86.7)
- added REF**: Via_GND_1, Additional:Via_GND_1, F.Cu at (160.5, 89.3)
- added REF**: Via_GND_04, Additional:Via_GND_06, F.Cu at (144.8, 117.3)
- added REF**: Via_GND_1, Additional:Via_GND_1, F.Cu at (159.3, 89.3)
- added REF**: Via_GND_04, Additional:Via_GND_04, F.Cu at (151.5, 91.6)
- added REF**: Via_GND_04, Additional:Via_GND_04, F.Cu at (146.7, 94.9)
- added REF**: Via_GND_04, Additional:Via_GND_04, F.Cu at (147.7, 95.6)
- added REF**: Via_GND_04, Additional:Via_GND_04, F.Cu at (157.0, 95.5)
- added REF**: Via_GND_04, Additional:Via_GND_04, F.Cu at (155.8, 95.5)
- added REF**: Via_GND_04, Additional:Via_GND_04, F.Cu at (154.7, 95.5)
- added REF**: Via_GND_04, Additional:Via_GND_04, F.Cu at (149.9, 95.1)
- added REF**: Via_GND_04, Additional:Via_GND_04, F.Cu at (148.3, 95.6)
- added REF**: Via_GND_04, Additional:Via_GND_04, F.Cu at (138.9, 115.6)
- added REF**: Via_GND_04, Additional:Via_GND_06, F.Cu at (143.9, 117.3)
- added REF**: Via_GND_04, Additional:Via_GND_04, F.Cu at (138.4, 116.7)
- added REF**: Via_GND_04, Additional:Via_GND_04, F.Cu at (154.6, 104.5)
- added REF**: Via_GND_04, Additional:Via_GND_04, F.Cu at (150.9, 104.1)
- added REF**: Via_GND_04, Additional:Via_GND_04, F.Cu at (178.4, 105.4)
- added REF**: Via_GND_04, Additional:Via_GND_04, F.Cu at (178.4, 104.5)
- added REF**: Via_GND_04, Additional:Via_GND_04, F.Cu at (176.8, 101.5)
- added REF**: Via_GND_04, Additional:Via_GND_04, F.Cu at (174.5, 101.7)
- added REF**: Via_GND_04, Additional:Via_GND_04, F.Cu at (174.5, 103.5)
- added REF**: Via_GND_04, Additional:Via_GND_04, F.Cu at (176.4, 108.7)
- added REF**: Via_GND_04, Additional:Via_GND_04, F.Cu at (176.4, 109.6)
- added REF**: Via_GND_04, Additional:Via_GND_06, F.Cu at (144.8, 116.5)
- added REF**: Via_GND_04, Additional:Via_GND_04, F.Cu at (170.9, 119.8)
- added REF**: Via_GND_04, Additional:Via_GND_04, F.Cu at (172.2, 119.8)
- added REF**: Via_GND_04, Additional:Via_GND_04, F.Cu at (173.5, 119.8)
- added REF**: Via_GND_04, Additional:Via_GND_04, F.Cu at (174.8, 119.8)
- added REF**: Via_GND_04, Additional:Via_GND_04, F.Cu at (176.3, 114.7)
- added REF**: Via_GND_04, Additional:Via_GND_04, F.Cu at (174.9, 114.7)
- added REF**: Via_GND_04, Additional:Via_GND_04, F.Cu at (166.1, 117.6)
- added REF**: Via_GND_04, Additional:Via_GND_04, F.Cu at (163.6, 119.5)
- added REF**: Via_GND_04, Additional:Via_GND_04, F.Cu at (163.6, 118.2)
- added REF**: Via_GND_04, Additional:Via_GND_04, F.Cu at (163.6, 117.0)
- added REF**: Via_GND_04, Additional:Via_GND_04, F.Cu at (161.4, 101.5)
- added REF**: Via_GND_04, Additional:Via_GND_04, F.Cu at (137.7, 116.1)
- added REF**: Via_GND_1, Additional:Via_GND_1, F.Cu at (175.9, 120.0)
- added REF**: Via_GND_1, Additional:Via_GND_1, F.Cu at (175.7, 107.8)
- added REF**: Via_GND_1, Additional:Via_GND_1, F.Cu at (160.5, 104.5)
- added REF**: Via_GND_1, Additional:Via_GND_1, F.Cu at (158.0, 101.1)
- added REF**: Via_GND_1, Additional:Via_GND_1, F.Cu at (158.0, 89.3)
- added REF**: Via_GND_1, Additional:Via_GND_1, F.Cu at (149.1, 109.5)
- added REF**: Via_GND_1, Additional:Via_GND_1, F.Cu at (138.0, 113.6)
- added REF**: Via_GND_1, Additional:Via_GND_1, F.Cu at (138.0, 110.3)
- added REF**: Via_GND_04, Additional:Via_GND_04, F.Cu at (162.6, 103.6)
- added REF**: Via_GND_04, Additional:Via_GND_06, F.Cu at (152.5, 104.2)
- added REF**: Via_GND_04, Additional:Via_GND_04, F.Cu at (137.7, 116.7)
- added REF**: Via_GND_04, Additional:Via_GND_04, F.Cu at (155.3, 101.3)
- added REF**: Via_GND_04, Additional:Via_GND_06, F.Cu at (143.9, 116.5)
- moved REF** 1.09 mm to (138.0, 111.9)
- moved C4 0.06 mm to (152.2, 99.5)
Routing:
- net Net-(R37-Pad1): track 30.0 -> 25.8 mm
- net V5: track 22.0 -> 23.9 mm
- net Net-(C4-Pad2): track 28.2 -> 26.6 mm
- net Net-(D10-Pad1): track 4.32 -> 2.73 mm
- net Net-(C12-Pad1): track 21.6 -> 22.3 mm
- net Net-(D7-Pad1): track 13.5 -> 12.9 mm
- net Net-(D8-Pad2): track 7.30 -> 7.67 mm, vias 3 -> 2
- net Net-(C2-Pad1): track 14.1 -> 14.3 mm, vias 0 -> 1
Other:
- rule trace_min: 0.1 -> 0.2

Commit message: Finished rev 1 and generated gerber files.
Parts:
- added REF**: Via_GND_04, Additional:Via_GND_04, F.Cu at (143.7, 109.7)
- added REF**: Via_GND_04, Additional:Via_GND_04, F.Cu at (152.0, 107.8)
- added REF**: Via_GND_04, Additional:Via_GND_04, F.Cu at (146.6, 106.0)
- added REF**: Via_GND_04, Additional:Via_GND_04, F.Cu at (146.6, 105.4)
- added REF**: Via_GND_04, Additional:Via_GND_04, F.Cu at (159.3, 95.8)
- added REF**: Via_GND_04, Additional:Via_GND_04, F.Cu at (159.3, 95.2)
- added REF**: Via_GND_04, Additional:Via_GND_04, F.Cu at (167.5, 107.6)
- added REF**: Via_GND_04, Additional:Via_GND_04, F.Cu at (170.1, 112.0)
- added REF**: Via_GND_04, Additional:Via_GND_04, F.Cu at (169.2, 108.6)
- added REF**: Via_GND_04, Additional:Via_GND_04, F.Cu at (170.2, 105.8)
- added REF**: Via_GND_04, Additional:Via_GND_04, F.Cu at (172.3, 105.8)
- added REF**: Via_GND_04, Additional:Via_GND_06, F.Cu at (145.9, 114.7)
- added REF**: Via_GND_04, Additional:Via_GND_04, F.Cu at (173.6, 105.8)
- added REF**: Via_GND_04, Additional:Via_GND_04, F.Cu at (160.7, 105.4)
- added REF**: Via_GND_04, Additional:Via_GND_04, F.Cu at (161.5, 103.6)
- added REF**: Via_GND_04, Additional:Via_GND_04, F.Cu at (155.7, 107.8)
- added REF**: Via_GND_04, Additional:Via_GND_04, F.Cu at (144.1, 106.8)
- added REF**: Via_GND_04, Additional:Via_GND_04, F.Cu at (143.6, 106.4)
- added REF**: Via_GND_04, Additional:Via_GND_04, F.Cu at (143.7, 109.1)
- added REF**: Via_GND_04, Additional:Via_GND_04, F.Cu at (141.6, 117.8)
- added REF**: Via_GND_04, Additional:Via_GND_04, F.Cu at (142.1, 115.9)
- added REF**: Via_GND_04, Additional:Via_GND_06, F.Cu at (143.9, 113.9)
- added REF**: Via_GND_04, Additional:Via_GND_04, F.Cu at (146.5, 116.7)
- added REF**: Via_GND_04, Additional:Via_GND_04, F.Cu at (158.5, 116.8)
- added REF**: Via_GND_04, Additional:Via_GND_04, F.Cu at (160.8, 118.6)
- added REF**: Via_GND_04, Additional:Via_GND_04, F.Cu at (144.4, 99.4)
- added REF**: Via_GND_04, Additional:Via_GND_04, F.Cu at (144.4, 91.6)
- added REF**: Via_GND_04, Additional:Via_GND_04, F.Cu at (146.7, 91.6)
- moved G*** 1.75 mm to (152.5, 112.3)
- renumbered W2 to W1, W3 to W2, W5 to W3, W1 to W5, W9 to W8, W8 to W9
Routing:
- net LED_GND: track 4.67 -> 7.02 mm
- net Net-(R33-Pad1): track 51.7 -> 52.2 mm
Other:
- board text added: "C22"
- board text added: "D10"
- board text added: "D11"
- board text added: "D2"
- board text added: "D4"
- board text added: "D6"
- board text added: "D7"
- board text added: "D8"
- board text added: "D9"
- board text added: "U3"

Commit message: Fixed a bug.
Parts:
- removed the REF** at (175.7, 107.8)
- added REF**: Via_GND_04, Additional:Via_GND_04, F.Cu at (176.5, 106.9)
- moved REF** 2.90 mm to (173.6, 108.0)
- moved REF** 2.08 mm to (175.1, 108.0)
- moved P3 1.00 mm to (164.0, 123.0)
Connections:
- P3 pad 2: LED_G -> LED_B
- P3 pad 3: LED_B -> LED_G
- R2 pad 2: Net-(C2-Pad1) -> V28
Routing:
- net LED_B: track 54.1 -> 70.5 mm, vias 4 -> 5
- net LED_G: track 50.7 -> 34.7 mm
- net V28: track 15.3 -> 28.7 mm
- net Net-(C2-Pad1): track 14.3 -> 7.30 mm

Commit message: Produced some output. Merge with master.
Parts:
- added REF**: Via_GND_04, Additional:Via_GND_04, F.Cu at (158.5, 123.3)
- added REF**: Via_GND_04, Additional:Via_GND_04, F.Cu at (158.5, 121.4)
- added REF**: Via_GND_04, Additional:Via_GND_04, F.Cu at (161.3, 121.4)
- added REF**: Via_GND_04, Additional:Via_GND_04, F.Cu at (161.3, 123.3)
- moved REF** 0.28 mm to (155.2, 100.6)
- moved REF** 0.13 mm to (155.2, 101.3)
Connections:
- U2 pad 5: Net-(C4-Pad2) -> V5
Routing:
- net LED_G: track 34.7 -> 51.2 mm
- net LED_B: track 70.5 -> 54.1 mm, vias 5 -> 4
- net V5: track 23.9 -> 34.1 mm
- net Net-(C4-Pad2): track 26.6 -> 25.1 mm
