File: pcb/power/bucketConvs.sch (KiCad schematic (older format))
At the start: 22 parts, among them U1 LM2840, U2 TS30012, U3 TPS2514ADBV

Commit message: Fixed a bug.
Parts:
- C2: Digikey 311-1088-1-ND -> 311-1343-1-ND
- R3: Digikey 311-10.0KHRCT-ND -> 311-10KGRCT-ND
- U1: Digikey LM2840XMK-ADJL/NOPBTR-ND -> LM2840XMK-ADJL/NOPBCT-ND
Connections:
- net V28: now also R2.2
- net at C2.1, D2.1 (K), L1.1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: no longer R2.2
Changed lines of the file:
@@
 F 2 "TO_SOT_Packages_SMD:SOT-23-6" H 2300 2550 60  0001 C CNN
 F 3 "http://www.ti.com/lit/ds/symlink/lm2841.pdf" H 2300 2550 60  0001 C CNN
-F 4 "LM2840XMK-ADJL/NOPBTR-ND" H 2300 2550 60  0001 C CNN "Digikey"
+F 4 "LM2840XMK-ADJL/NOPBCT-ND" H 2300 2550 60  0001 C CNN "Digikey"
 	1    2300 2550
 	1    0    0    -1
@@
 F 2 "Capacitors_SMD:C_0603_HandSoldering" H 2338 1950 50  0001 C CNN
 F 3 "http://www.yageo.com/documents/recent/UPY-GPHC_X7R_6.3V-to-50V_15.pdf" H 2300 2100 50  0001 C CNN
-F 4 "311-1088-1-ND" H 2300 2100 60  0001 C CNN "Digikey"
+F 4 "311-1343-1-ND" H 2300 2100 60  0001 C CNN "Digikey"
 	1    2300 2100
 	0    1    1    0
 $EndComp
 $Comp
-L GND #PWR5
+L GND #PWR07
 U 1 1 5842EC4A
 P 1700 2550
-F 0 "#PWR5" H 1700 2300 50  0001 C CNN
+F 0 "#PWR07" H 1700 2300 50  0001 C CNN
 F 1 "GND" H 1700 2400 50  0000 C CNN
 F 2 "" H 1700 2550 50  0000 C CNN
@@
 $EndComp
 $Comp
-L GND #PWR7
+L GND #PWR08
 U 1 1 5842EC58
 P 3000 3600
-F 0 "#PWR7" H 3000 3350 50  0001 C CNN
+F 0 "#PWR08" H 3000 3350 50  0001 C CNN
 F 1 "GND" H 3000 3450 50  0000 C CNN
 F 2 "" H 3000 3600 50  0000 C CNN
@@
 F 2 "Additional:R_0603_HandSoldering_Same_As_C" V 1730 2950 50  0001 C CNN
 F 3 "http://www.yageo.com.tw/exep/pages/download/literatures/PYu-R_INT-thick_7.pdf" H 1800 2950 50  0001 C CNN
-F 4 " 311-10.0KHRCT-ND" V 1800 2950 60  0001 C CNN "Digikey"
+F 4 "311-10KGRCT-ND" V 1800 2950 60  0001 C CNN "Digikey"
 	1    1800 2950
 	1    0    0    -1
@@
 $EndComp
 $Comp
-L GND #PWR6
+L GND #PWR09
 U 1 1 5842F8AB
 P 1800 5650
-F 0 "#PWR6" H 1800 5400 50  0001 C CNN
+F 0 "#PWR09" H 1800 5400 50  0001 C CNN
 F 1 "GND" H 1800 5500 50  0000 C CNN
 F 2 "" H 1800 5650 50  0000 C CNN
@@
 5V for Mobile Phone\n-----------------------\nVout,max=5 V\nAout,max = 2A
 $Comp
-L GND #PWR8
+L GND #PWR010
 U 1 1 5842F939
 P 4100 5200
-F 0 "#PWR8" H 4100 4950 50  0001 C CNN
+F 0 "#PWR010" H 4100 4950 50  0001 C CNN
 F 1 "GND" H 4100 5050 50  0000 C CNN
 F 2 "" H 4100 5200 50  0000 C CNN
@@
 $EndComp
 $Comp
-L PWR_FLAG #FLG3
+L PWR_FLAG #FLG011
 U 1 1 5842F941
 P 5750 5250
-F 0 "#FLG3" H 5750 5345 50  0001 C CNN
+F 0 "#FLG011" H 5750 5345 50  0001 C CNN
 F 1 "PWR_FLAG" H 5750 5430 50  0000 C CNN
 F 2 "" H 5750 5250 50  0000 C CNN
@@
 	0    -1   -1   0
 $EndComp
-Wire Wire Line
-	2800 2400 3700 2400
-Wire Wire Line
-	1800 2400 1800 2100
-Wire Wire Line
-	1800 2100 2150 2100
-Wire Wire Line
-	2450 2100 2850 2100
-Wire Wire Line
-	2850 2100 2850 2400
-Connection ~ 2850 2400
-Wire Wire Line
-	3650 1950 3650 2775
-Connection ~ 3650 2400
-Wire Wire Line
-	4350 2400 4350 2750
-Wire Wire Line
-	3650 3550 3650 3075
-Connection ~ 4350 2400
-Wire Wire Line
-	1700 2550 1800 2550
-Wire Wire Line
-	2800 2700 2900 2700
-Wire Wire Line
-	2900 2700 2900 2550
-Connection ~ 2900 2550
-Wire Wire Line
-	3000 3000 3000 3600
-Wire Wire Line
-	3000 2550 3000 2700
-Wire Wire Line
-	1800 3150 1800 3100
-Wire Wire Line
-	1800 2700 1800 2800
-Wire Wire Line
-	1800 2750 1600 2750
-Connection ~ 1800 2750
-Wire Wire Line
-	1200 2750 1200 1950
-Wire Wire Line
-	1200 1950 3650 1950
-Wire Wire Line
-	1200 2750 1300 2750
-Connection ~ 3000 3550
-Wire Wire Line
-	1800 3550 1800 3450
-Wire Wire Line
-	2800 2550 3150 2550
-Wire Wire Line
-	4800 2900 4800 2850
-Wire Wire Line
-	4800 3550 4800 3200
-Wire Wire Line
-	4800 2400 4800 2450
-Connection ~ 4350 3550
-Connection ~ 3000 2550
-Wire Wire Line
-	1800 5250 1800 5200
-Connection ~ 1800 5200
-Wire Wire Line
-	1800 5550 1800 5650
-Connection ~ 1800 5600
-Wire Wire Line
-	3900 5400 4950 5400
-Connection ~ 5750 5400
-Wire Wire Line
-	4850 5500 4850 5400
-Connection ~ 4850 5400
-Wire Wire Line
-	5750 5250 5750 5500
-Wire Wire Line
-	6200 5400 6200 5500
-Wire Wire Line
-	4850 5800 4850 6300
-Wire Wire Line
-	6200 6300 6200 5800
-Wire Wire Line
-	5750 5800 5750 6300
-Connection ~ 5750 6300
-Wire Wire Line
-	1650 5200 2300 5200
-Wire Wire Line
-	2300 5400 2000 5400
-Wire Wire Line
-	2000 5400 2000 5600
-Wire Wire Line
-	2000 5600 1800 5600
-Wire Wire Line
-	3900 5600 4100 5600
-Connection ~ 4550 5400
-Wire Wire Line
-	2300 5600 2150 5600
-Wire Wire Line
-	2150 5600 2150 6300
-Wire Wire Line
-	4700 6300 4700 5400
-Connection ~ 4700 5400
-Connection ~ 6200 5400
-Wire Wire Line
-	4100 5800 3900 5800
-Wire Wire Line
-	4550 5600 4400 5600
-Wire Wire Line
-	6600 5850 6600 5950
-Wire Wire Line
-	6600 5400 6600 5450
-Wire Wire Line
-	6600 6250 6600 6350
-Connection ~ 6200 6300
-Wire Wire Line
-	3900 5200 4100 5200
-Wire Wire Line
-	4550 5400 4550 5600
-Wire Wire Line
-	5550 5400 6850 5400
-Wire Wire Line
-	2150 6300 4700 6300
-Wire Wire Line
-	4850 6300 6600 6300
-Wire Wire Line
-	1800 3550 4800 3550
-Wire Wire Line
-	4300 2400 5150 2400
-Connection ~ 6600 5400
-Connection ~ 4800 2400
-$Comp
-L GND #PWR9
+$Comp
+L GND #PWR012
 U 1 1 584C8E69
 P 6600 6350
-F 0 "#PWR9" H 6600 6100 50  0001 C CNN
+F 0 "#PWR012" H 6600 6100 50  0001 C CNN
 F 1 "GND" H 6600 6200 50  0000 C CNN
 F 2 "" H 6600 6350 50  0000 C CNN
@@
 	1    0    0    -1
 $EndComp
-Connection ~ 6600 6300
 $Comp
 L TPS2514ADBV U3
@@
 V5
 $Comp
-L GND #PWR10
+L GND #PWR013
 U 1 1 5865A9E7
 P 7350 3500
-F 0 "#PWR10" H 7350 3250 50  0001 C CNN
+F 0 "#PWR013" H 7350 3250 50  0001 C CNN
 F 1 "GND" H 7350 3350 50  0000 C CNN
 F 2 "" H 7350 3500 50  0000 C CNN
@@
 	1    0    0    -1
 $EndComp
-Wire Wire Line
-	7350 3500 7400 3500
 Text Notes 7000 4550 0    60   ~ 0
 USB Dedicated Charging Port Control.\n-----------------------\nSimple SOT-23-6 IC for detecting propriatary and open standards used by a\ndevice and providing the corresponding electrical signature at the data lines\n(voltage or impedance).
 Text HLabel 8450 3300 2    60   Output ~ 0
 DM1
-Wire Wire Line
-	8400 3300 8450 3300
 Text HLabel 7350 3300 0    60   Output ~ 0
 DP1
-Wire Wire Line
-	7400 3300 7350 3300
 $Comp
 L C C22
@@
 	1    0    0    -1
 $EndComp
-Wire Wire Line
-	8400 3500 8850 3500
-Connection ~ 8650 3500
-$Comp
-L GND #PWR11
+$Comp
+L GND #PWR014
 U 1 1 58662C1C
 P 8650 3800
-F 0 "#PWR11" H 8650 3550 50  0001 C CNN
+F 0 "#PWR014" H 8650 3550 50  0001 C CNN
 F 1 "GND" H 8650 3650 50  0000 C CNN
 F 2 "" H 8650 3800 50  0000 C CNN
@@
 NoConn ~ 3100 6050
 Wire Wire Line
+	2800 2400 3700 2400
+Wire Wire Line
+	1800 2400 1800 2100
+Wire Wire Line
+	1800 2100 2150 2100
+Wire Wire Line
+	2450 2100 2850 2100
+Wire Wire Line
+	2850 2100 2850 2400
+Connection ~ 2850 2400
+Connection ~ 3650 2400
+Wire Wire Line
+	4350 1950 4350 2750
+Wire Wire Line
+	3650 3550 3650 3075
+Connection ~ 4350 2400
+Wire Wire Line
+	1700 2550 1800 2550
+Wire Wire Line
+	2800 2700 2900 2700
+Wire Wire Line
+	2900 2700 2900 2550
+Connection ~ 2900 2550
+Wire Wire Line
+	3000 3000 3000 3600
+Wire Wire Line
+	3000 2550 3000 2700
+Wire Wire Line
+	1800 3150 1800 3100
+Wire Wire Line
+	1800 2700 1800 2800
+Wire Wire Line
+	1800 2750 1600 2750
+Connection ~ 1800 2750
+Wire Wire Line
+	1200 2750 1200 1950
+Wire Wire Line
+	1200 2750 1300 2750
+Connection ~ 3000 3550
+Wire Wire Line
+	1800 3550 1800 3450
+Wire Wire Line
+	2800 2550 3150 2550
+Wire Wire Line
+	4800 2900 4800 2850
+Wire Wire Line
+	4800 3550 4800 3200
+Wire Wire Line
+	4800 2400 4800 2450
+Connection ~ 4350 3550
+Connection ~ 3000 2550
+Wire Wire Line
+	1800 5250 1800 5200
+Connection ~ 1800 5200
+Wire Wire Line
+	1800 5550 1800 5650
+Connection ~ 1800 5600
+Wire Wire Line
+	3900 5400 4950 5400
+Connection ~ 5750 5400
+Wire Wire Line
+	4850 5500 4850 5400
+Connection ~ 4850 5400
+Wire Wire Line
+	5750 5250 5750 5500
+Wire Wire Line
+	6200 5400 6200 5500
+Wire Wire Line
+	4850 5800 4850 6300
+Wire Wire Line
+	6200 6300 6200 5800
+Wire Wire Line
+	5750 5800 5750 6300
+Connection ~ 5750 6300
+Wire Wire Line
+	1650 5200 2300 5200
+Wire Wire Line
+	2300 5400 2000 5400
+Wire Wire Line
+	2000 5400 2000 5600
+Wire Wire Line
+	2000 5600 1800 5600
+Wire Wire Line
+	3900 5600 4100 5600
+Connection ~ 4550 5400
+Wire Wire Line
+	2300 5600 2150 5600
+Wire Wire Line
+	2150 5600 2150 6300
+Wire Wire Line
+	4700 6300 4700 5400
+Connection ~ 4700 5400
+Connection ~ 6200 5400
+Wire Wire Line
+	4100 5800 3900 5800
+Wire Wire Line
+	4550 5600 4400 5600
+Wire Wire Line
+	6600 5850 6600 5950
+Wire Wire Line
+	6600 5400 6600 5450
+Wire Wire Line
+	6600 6250 6600 6350
+Connection ~ 6200 6300
+Wire Wire Line
+	3900 5200 4100 5200
+Wire Wire Line
+	4550 5400 4550 5600
+Wire Wire Line
+	5550 5400 6850 5400
+Wire Wire Line
+	2150 6300 4700 6300
+Wire Wire Line
+	4850 6300 6600 6300
+Wire Wire Line
+	1800 3550 4800 3550
+Wire Wire Line
+	4300 2400 5150 2400
+Connection ~ 6600 5400
+Connection ~ 4800 2400
+Connection ~ 6600 6300
+Wire Wire Line
+	7350 3500 7400 3500
+Wire Wire Line
+	8400 3300 8450 3300
+Wire Wire Line
+	7400 3300 7350 3300
+Wire Wire Line
+	8400 3500 8850 3500
+Connection ~ 8650 3500
+Wire Wire Line
 	4350 3550 4350 3050
 Connection ~ 3650 3550
+Wire Wire Line
+	3650 2400 3650 2775
+Wire Wire Line
+	1200 1950 4350 1950
 $EndSCHEMATC

Commit message: Produced some output. Merge with master.
Connections:
- net V5: now also U2.5 (FB)
- net at C4.2, D4.1 (K), L2.1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: no longer U2.5 (FB)
Changed lines of the file:
@@
 	1    0    0    -1
 $EndComp
-Text Notes 1200 1900 0    60   ~ 0
+Text Notes 1175 1375 0    60   ~ 0
 2.8 V for µC\n---------------------------\nVout=0.765 V (1 + (27k/ 10.15k))=2.8 V\n27k/10.15k= 2.66
 $Comp
@@
 	1    0    0    -1
 $EndComp
-Text Notes 1400 5000 0    60   ~ 0
+Text Notes 1325 4875 0    60   ~ 0
 5V for Mobile Phone\n-----------------------\nVout,max=5 V\nAout,max = 2A
 $Comp
@@
 	5750 5250 5750 5500
 Wire Wire Line
-	6200 5400 6200 5500
+	6200 4925 6200 5500
 Wire Wire Line
 	4850 5800 4850 6300
@@
 	3900 5600 4100 5600
 Connection ~ 4550 5400
-Wire Wire Line
-	2300 5600 2150 5600
-Wire Wire Line
-	2150 5600 2150 6300
-Wire Wire Line
-	4700 6300 4700 5400
-Connection ~ 4700 5400
 Connection ~ 6200 5400
 Wire Wire Line
@@
 Wire Wire Line
 	5550 5400 6850 5400
-Wire Wire Line
-	2150 6300 4700 6300
 Wire Wire Line
 	4850 6300 6600 6300
@@
 Wire Wire Line
 	1200 1950 4350 1950
+Wire Wire Line
+	6200 4925 1325 4925
+Wire Wire Line
+	1325 4925 1325 5900
+Wire Wire Line
+	2300 5600 2150 5600
+Wire Wire Line
+	2150 5600 2150 5900
+Wire Wire Line
+	2150 5900 1325 5900
 $EndSCHEMATC

Commit message: Minor changes.
Parts:
- D3, D5: symbol LED -> LED-RESCUE-power
Changed lines of the file:
@@
 EESchema Schematic File Version 2
+LIBS:power-rescue
 LIBS:power
 LIBS:device
@@
 $EndComp
 $Comp
-L LED D3
+L LED-RESCUE-power D3
 U 1 1 5842EC88
 P 4800 2650
@@
 $EndComp
 $Comp
-L LED D5
+L LED-RESCUE-power D5
 U 1 1 5842F8E3
 P 6600 5650
